Commit message: finished desing of roobot

File: diff_drive/urdf/ddrive.urdf.xacro (robot description, xacro)
@@ -1,4 +1,4 @@
 <?xml version="1.0"?>
-<robot xmlns:xacro="http://www.ros.org/wiki/xacro" name="slidebot">
+<robot name="myRobot" xmlns:xacro="http://www.ros.org/wiki/xacro">
 <xacro:include filename="$(find diff_drive)/urdf/materials.xacro"/>
 <xacro:property name="yaml_file" value="$(find diff_drive)/config/robo_parameters.yaml" />
@@ -21,6 +21,20 @@
         </visual>
     </link>
-    <joint name="joint_${link_name}" type="fixed">
-        <parent link="base"/>
+    <collision>
+      <geometry>
+        <cylinder radius="${2*height}" length="${length_wheel}" />
+        <origin xyz="0.0 ${L_R*length_wheel/2} 0.0" rpy="${pi/2} 0 0" />
+      </geometry>
+    </collision>
+    <inertial>
+      <origin xyz="0.0 ${L_R*length_wheel/2} 0.0" rpy="${pi/2} 0 0" />
+      <mass value="0.5"/>
+      <inertia
+        ixx="${1/12*0.5*(3*4*height*height+length_wheel*length_wheel)}" ixy="0.0" ixz="0.0"
+        iyy="${1/12*0.5*(3*4*height*height+length_wheel*length_wheel)}" iyz="0.0"
+        izz="${0.5*0.5*4*height*height}"/>
+    </inertial>
+    <joint name="joint_${link_name}" type="continuous">
+        <parent link="base_robot"/>
         <child link="${link_name}"/>
         <origin xyz="${length/2} ${L_R*width/2} 0.0" rpy="0 0 0"/>
@@ -28,6 +42,15 @@
     </joint>
 </xacro:macro>
-<!-- visual for my base frame -->
-  <link name="base">
+<link name="base">
+  <visual>
+    <geometry>
+      <box size="0.1 0.1 0.1"/>
+    </geometry>
+    <origin rpy="0 0 0" xyz="0 0 0"/>
+    <material name="green"/>
+  </visual>
+</link>
+<!-- visual for my base_robot frame -->
+  <link name="base_robot">
     <visual>
       <geometry>
@@ -37,4 +60,16 @@
       <material name="green"/>
     </visual>
+    <collision>
+      <geometry>
+        <box size="${length} ${width} ${height}"/>
+      </geometry>
+    </collision>
+    <inertial>
+      <mass value="1.0"/>
+      <inertia
+        ixx="${1/12*1*(length*length+width*width)}" ixy="0.0" ixz="0.0"
+        iyy="${1/12*1*(width*width+height*height)}"  iyz="0.0"
+        izz="${1/12*1*(length*length+height*height)}" />
+    </inertial>
     <collision name='caster_up_collision'>
         <origin xyz="${-length*3/8} 0 ${height}" rpy=" 0 0 0"/>
@@ -58,5 +93,5 @@
             <sphere radius="${height/2}"/>
         </geometry>
-        <material name="yellow"/>
+        <material name="brown"/>
     </visual>
     <collision name='caster_down_collision'>
@@ -81,5 +116,5 @@
             <sphere radius="${height/2}"/>
         </geometry>
-        <material name="yellow"/>
+        <material name="brown"/>
     </visual>
   </link>
@@ -97,15 +132,36 @@
       </geometry>
       <origin xyz="0.0 0 ${length*2/3}" rpy="0 0 0" />
-      <material name="yellow"/>
+      <material name="brown"/>
     </visual>
+    <collision>
+      <geometry>
+        <box size="${flipper_size} ${flipper_size} ${length*2/3}"/>
+        <origin xyz="0.0 0 ${length*2/6}" rpy="0 0 0" />
+      </geometry>
+    </collision>
+    <inertial>
+      <origin xyz="0.0 0 ${length*2/6}" rpy="0 0 0" />
+      <mass value="2.0"/>
+      <inertia
+        ixx="${1/3*2*length*2/3*length*2/3}" ixy="0.0" ixz="0.0"
+        iyy="0.0" iyz="0.0"
+        izz="${1/3*2*length*2/3*length*2/3}"/>
+    </inertial>
   </link>
   <joint name="joint_flipper" type="continuous">
-    <parent link="base"/>
+    <parent link="base_robot"/>
     <child link="flipper"/>
     <origin xyz="${length/2+flipper_size/2} 0 0.0" rpy="0 0 0"/>
     <axis xyz="0 1 0"/>
   </joint>
+  <joint name="joint_base_to_base" type="fixed">
+    <parent link="base"/>
+    <child link="base_robot"/>
+    <origin xyz="0 0 0.0" rpy="0 0 0"/>
+    <!-- <axis xyz="0 1 0"/> -->
+  </joint>
   <!-- create wheels -->
-  <xacro:wheel link_name="left_wheel"  joint_parent="base" L_R="1.0"/>
-  <xacro:wheel link_name="right_wheel" joint_parent="base" L_R="-1.0"/>
+  <xacro:wheel link_name="left_wheel"  joint_parent="base_robot" L_R="1.0"/>
+  <xacro:wheel link_name="right_wheel" joint_parent="base_robot" L_R="-1.0"/>
   </robot>
+<!-- https://github.com/Geekgineer/spcbot/blob/master/spcbot_description/urdf/materials.xacro -->

Commit message: switching my robot

File: diff_drive/urdf/ddrive.urdf.xacro (robot description, xacro)
@@ -1,81 +1,35 @@
-<?xml version="1.0"?>
-<robot name="myRobot" xmlns:xacro="http://www.ros.org/wiki/xacro">
-<xacro:include filename="$(find diff_drive)/urdf/materials.xacro"/>
-<xacro:property name="yaml_file" value="$(find diff_drive)/config/robo_parameters.yaml" />
-<xacro:property name="props"  value="${load_yaml(yaml_file)}"/>
-<xacro:property name="scale"  value="${props['scale']}" />
-<xacro:property name="width"  value="${props['width' ]*scale}" />
-<xacro:property name="height" value="${props['height']*scale}" />
-<xacro:property name="length" value="${props['length']*scale}" />
-<xacro:property name="length_wheel" value="${props['length_wheel']*scale}" />
-<xacro:property name="flipper_size" value="${props['flipper_size']*scale}" />
-<!-- create wheels  -->
-<xacro:macro name="wheel" params="link_name joint_parent L_R">
-    <link name="${link_name}">
-        <visual>
-            <geometry>
-                <cylinder radius="${2*height}" length="${length_wheel}" />
-            </geometry>
-            <origin xyz="0.0 ${L_R*length_wheel/2} 0.0" rpy="${pi/2} 0 0" />
-            <material name="red"/>
-        </visual>
-    </link>
-    <collision>
+<?xml version="1.0" ?>
+<robot name="m2wr" xmlns:xacro="http://www.ros.org/wiki/xacro">
+  <xacro:include filename="$(find diff_drive)/urdf/materials.xacro" />
+  <xacro:include filename="$(find diff_drive)/urdf/ddrive.gazebo" />
+  <xacro:include filename="$(find diff_drive)/urdf/macros.xacro" />
+  <link name="link_chassis">
+    <!-- pose and inertial -->
+    <pose>0 0 0.1 0 0 0</pose>
+    <inertial>
+      <mass value="5"/>
+      <origin rpy="0 0 0" xyz="0 0 0.1"/>
+      <inertia ixx="0.0395416666667" ixy="0" ixz="0" iyy="0.106208333333" iyz="0" izz="0.106208333333"/>
+    </inertial>
+    <!-- body -->
+    <collision name="collision_chassis">
       <geometry>
-        <cylinder radius="${2*height}" length="${length_wheel}" />
-        <origin xyz="0.0 ${L_R*length_wheel/2} 0.0" rpy="${pi/2} 0 0" />
+        <box size="0.5 0.3 0.07"/>
       </geometry>
     </collision>
-    <inertial>
-      <origin xyz="0.0 ${L_R*length_wheel/2} 0.0" rpy="${pi/2} 0 0" />
-      <mass value="0.5"/>
-      <inertia
-        ixx="${1/12*0.5*(3*4*height*height+length_wheel*length_wheel)}" ixy="0.0" ixz="0.0"
-        iyy="${1/12*0.5*(3*4*height*height+length_wheel*length_wheel)}" iyz="0.0"
-        izz="${0.5*0.5*4*height*height}"/>
-    </inertial>
-    <joint name="joint_${link_name}" type="continuous">
-        <parent link="base_robot"/>
-        <child link="${link_name}"/>
-        <origin xyz="${length/2} ${L_R*width/2} 0.0" rpy="0 0 0"/>
-        <axis xyz="0 1 0" rpy="0 0 0"/>
-    </joint>
-</xacro:macro>
-<link name="base">
-  <visual>
-    <geometry>
-      <box size="0.1 0.1 0.1"/>
-    </geometry>
-    <origin rpy="0 0 0" xyz="0 0 0"/>
-    <material name="green"/>
-  </visual>
-</link>
-<!-- visual for my base_robot frame -->
-  <link name="base_robot">
     <visual>
+      <origin rpy="0 0 0" xyz="0 0 0"/>
       <geometry>
-        <box size="${length} ${width} ${height}"/>
+        <box size="0.5 0.3 0.07"/>
       </geometry>
-      <origin rpy="0 0 0" xyz="0 0 0"/>
-      <material name="green"/>
+      <material name="blue"/>
     </visual>
-    <collision>
+    <!-- caster front -->
+    <collision name="caster_front_collision">
+      <origin rpy=" 0 0 0" xyz="0.35 0 -0.05"/>
       <geometry>
-        <box size="${length} ${width} ${height}"/>
+        <sphere radius="0.05"/>
       </geometry>
-    </collision>
-    <inertial>
-      <mass value="1.0"/>
-      <inertia
-        ixx="${1/12*1*(length*length+width*width)}" ixy="0.0" ixz="0.0"
-        iyy="${1/12*1*(width*width+height*height)}"  iyz="0.0"
-        izz="${1/12*1*(length*length+height*height)}" />
-    </inertial>
-    <collision name='caster_up_collision'>
-        <origin xyz="${-length*3/8} 0 ${height}" rpy=" 0 0 0"/>
-        <geometry>
-            <sphere radius="${height/2}"/>
-      </geometry>
-      <!-- <surface>
+      <surface>
         <friction>
           <ode>
@@ -86,82 +40,41 @@
           </ode>
         </friction>
-      </surface> -->
+      </surface>
     </collision>
-    <visual name='caster_up_visual'>
-        <origin xyz="${-length*3/8} 0 ${height}" rpy=" 0 0 0"/>
-        <geometry>
-            <sphere radius="${height/2}"/>
-        </geometry>
-        <material name="brown"/>
-    </visual>
-    <collision name='caster_down_collision'>
-        <origin xyz="${-length*3/8} 0 -${height}" rpy=" 0 0 0"/>
-        <geometry>
-            <sphere radius="${height/2}"/>
-        </geometry>
-      <!-- <surface>
-        <friction>
-          <ode>
-            <mu>0</mu>
-            <mu2>0</mu2>
-            <slip1>1.0</slip1>
-            <slip2>1.0</slip2>
-          </ode>
-        </friction>
-      </surface> -->
-    </collision>
-    <visual name='caster_down_visual'>
-        <origin xyz="${-length*3/8} 0 -${height}" rpy=" 0 0 0"/>
-        <geometry>
-            <sphere radius="${height/2}"/>
-        </geometry>
-        <material name="brown"/>
+    <visual name="caster_front_visual">
+      <origin rpy=" 0 0 0" xyz="0.2 0 -0.05"/>
+      <geometry>
+        <sphere radius="0.05"/>
+      </geometry>
     </visual>
   </link>
-<link name="flipper">
+  <link name="sensor_laser">
+    <inertial>
+      <origin xyz="0 0 0" rpy="0 0 0" />
+      <mass value="1" />
+      <xacro:cylinder_inertia mass="1" r="0.05" l="0.1" />
+    </inertial>
     <visual>
+      <origin xyz="0 0 0" rpy="0 0 0" />
       <geometry>
-        <box size="${flipper_size} ${flipper_size} ${length*2/3}"/>
+        <cylinder radius="0.05" length="0.1"/>
       </geometry>
-      <origin xyz="0.0 0 ${length*2/6}" rpy="0 0 0" />
-      <material name="blue"/>
-    </visual>
-    <visual>
-      <geometry>
-        <sphere radius="${height/2}"/>
-      </geometry>
-      <origin xyz="0.0 0 ${length*2/3}" rpy="0 0 0" />
-      <material name="brown"/>
+      <material name="white" />
     </visual>
     <collision>
+      <origin xyz="0 0 0" rpy="0 0 0"/>
       <geometry>
-        <box size="${flipper_size} ${flipper_size} ${length*2/3}"/>
-        <origin xyz="0.0 0 ${length*2/6}" rpy="0 0 0" />
+        <cylinder radius="0.05" length="0.1"/>
       </geometry>
     </collision>
-    <inertial>
-      <origin xyz="0.0 0 ${length*2/6}" rpy="0 0 0" />
-      <mass value="2.0"/>
-      <inertia
-        ixx="${1/3*2*length*2/3*length*2/3}" ixy="0.0" ixz="0.0"
-        iyy="0.0" iyz="0.0"
-        izz="${1/3*2*length*2/3*length*2/3}"/>
-    </inertial>
   </link>
-  <joint name="joint_flipper" type="continuous">
-    <parent link="base_robot"/>
-    <child link="flipper"/>
-    <origin xyz="${length/2+flipper_size/2} 0 0.0" rpy="0 0 0"/>
-    <axis xyz="0 1 0"/>
+  <joint name="joint_sensor_laser" type="fixed">
+    <origin xyz="0.15 0 0.05" rpy="0 0 0"/>
+    <parent link="link_chassis"/>
+    <child link="sensor_laser"/>
   </joint>
-  <joint name="joint_base_to_base" type="fixed">
-    <parent link="base"/>
-    <child link="base_robot"/>
-    <origin xyz="0 0 0.0" rpy="0 0 0"/>
-    <!-- <axis xyz="0 1 0"/> -->
-  </joint>
-  <!-- create wheels -->
-  <xacro:wheel link_name="left_wheel"  joint_parent="base_robot" L_R="1.0"/>
-  <xacro:wheel link_name="right_wheel" joint_parent="base_robot" L_R="-1.0"/>
-  </robot>
-<!-- https://github.com/Geekgineer/spcbot/blob/master/spcbot_description/urdf/materials.xacro -->
+  <xacro:link_wheel name="link_right_wheel" />
+  <xacro:joint_wheel name="joint_right_wheel" child="link_right_wheel" origin_xyz="-0.05 0.20 0" />
+  <xacro:link_wheel name="link_left_wheel" />
+  <xacro:joint_wheel name="joint_left_wheel" child="link_left_wheel" origin_xyz="-0.05 -0.20 0" />
+</robot>

Commit message: working on following rectangle trajectory

File: diff_drive/urdf/ddrive.urdf.xacro (robot description, xacro)
@@ -49,29 +49,4 @@
     </visual>
   </link>
-  <link name="sensor_laser">
-    <inertial>
-      <origin xyz="0 0 0" rpy="0 0 0" />
-      <mass value="1" />
-      <xacro:cylinder_inertia mass="1" r="0.05" l="0.1" />
-    </inertial>
-    <visual>
-      <origin xyz="0 0 0" rpy="0 0 0" />
-      <geometry>
-        <cylinder radius="0.05" length="0.1"/>
-      </geometry>
-      <material name="white" />
-    </visual>
-    <collision>
-      <origin xyz="0 0 0" rpy="0 0 0"/>
-      <geometry>
-        <cylinder radius="0.05" length="0.1"/>
-      </geometry>
-    </collision>
-  </link>
-  <joint name="joint_sensor_laser" type="fixed">
-    <origin xyz="0.15 0 0.05" rpy="0 0 0"/>
-    <parent link="link_chassis"/>
-    <child link="sensor_laser"/>
-  </joint>
   <xacro:link_wheel name="link_right_wheel" />
   <xacro:joint_wheel name="joint_right_wheel" child="link_right_wheel" origin_xyz="-0.05 0.20 0" />

Commit message: added robot parameters yaml and second caster

File: diff_drive/urdf/ddrive.urdf.xacro (robot description, xacro)
@@ -4,4 +4,10 @@
   <xacro:include filename="$(find diff_drive)/urdf/ddrive.gazebo" />
   <xacro:include filename="$(find diff_drive)/urdf/macros.xacro" />
+<xacro:property name="robo_parameters" value="$(find diff_drive)/config/robo_parameters.yaml" />
+<xacro:property name="props" value="${load_yaml(robo_parameters)}"/>
+<xacro:property name="width" value="${props['width']}" />
+<xacro:property name="length" value="${props['length']}" />
+<xacro:property name="height" value="${props['height']}" />
+<xacro:property name="caster_radius" value="${props['caster_radius']}" />
   <link name="link_chassis">
     <!-- pose and inertial -->
@@ -15,5 +21,5 @@
     <collision name="collision_chassis">
       <geometry>
-        <box size="0.5 0.3 0.07"/>
+        <box size="${width} ${length} ${height}"/>
       </geometry>
     </collision>
@@ -21,13 +27,13 @@
       <origin rpy="0 0 0" xyz="0 0 0"/>
       <geometry>
-        <box size="0.5 0.3 0.07"/>
+        <box size="${width} ${length} ${height}"/>
       </geometry>
       <material name="blue"/>
     </visual>
-    <!-- caster front -->
-    <collision name="caster_front_collision">
+    <!-- caster down -->
+    <collision name="caster_down_collision">
       <origin rpy=" 0 0 0" xyz="0.35 0 -0.05"/>
       <geometry>
-        <sphere radius="0.05"/>
+        <sphere radius="${caster_radius}"/>
       </geometry>
       <surface>
@@ -42,8 +48,31 @@
       </surface>
     </collision>
-    <visual name="caster_front_visual">
+    <visual name="caster_down_visual">
       <origin rpy=" 0 0 0" xyz="0.2 0 -0.05"/>
       <geometry>
-        <sphere radius="0.05"/>
+        <sphere radius="${caster_radius}"/>
+      </geometry>
+    </visual>
+    <!-- caster up -->
+    <collision name="caster_up_collision">
+      <origin rpy=" 0 0 0" xyz="0.35 0 0.05"/>
+      <geometry>
+        <sphere radius="${caster_radius}"/>
+      </geometry>
+      <surface>
+        <friction>
+          <ode>
+            <mu>0</mu>
+            <mu2>0</mu2>
+            <slip1>1.0</slip1>
+            <slip2>1.0</slip2>
+          </ode>
+        </friction>
+      </surface>
+    </collision>
+    <visual name="caster_up_visual">
+      <origin rpy=" 0 0 0" xyz="0.2 0 0.05"/>
+      <geometry>
+        <sphere radius="${caster_radius}"/>
       </geometry>
     </visual>

Commit message: added dump variable,some more parameters

File: diff_drive/urdf/ddrive.urdf.xacro (robot description, xacro)
@@ -1,4 +1,4 @@
 <?xml version="1.0" ?>
-<robot name="m2wr" xmlns:xacro="http://www.ros.org/wiki/xacro">
+<robot name="my_diff_robot" xmlns:xacro="http://www.ros.org/wiki/xacro">
   <xacro:include filename="$(find diff_drive)/urdf/materials.xacro" />
   <xacro:include filename="$(find diff_drive)/urdf/ddrive.gazebo" />
@@ -10,4 +10,23 @@
 <xacro:property name="height" value="${props['height']}" />
 <xacro:property name="caster_radius" value="${props['caster_radius']}" />
+  <!-- <link name="World">
+      <visual>
+      <origin rpy="0 0 0" xyz="0 0 0"/>
+      <geometry>
+        <box size="${width} ${length} ${height}"/>
+      </geometry>
+    </visual>
+  </link>
+  <joint name="World_Joint" type="fixed">
+  <origin rpy="0 0 0" xyz="0 0 0"/>
+  <child link="link_chassis"/>
+  <parent link="World"/>
+  </joint> -->
+<link name="dummy">
+   </link>
+  <joint name="dummy_joint" type="fixed">
+     <parent link="dummy"/>
+     <child link="link_chassis"/>
+   </joint>
   <link name="link_chassis">
     <!-- pose and inertial -->

File: diff_drive/urdf/macros.xacro (robot description, xacro)
@@ -1,8 +1,13 @@
 <?xml version="1.0"?>
 <robot xmlns:xacro="http://www.ros.org/wiki/xacro">
+    <xacro:property name="robo_parameters" value="$(find diff_drive)/config/robo_parameters.yaml" />
+    <xacro:property name="props" value="${load_yaml(robo_parameters)}"/>
+    <xacro:property name="wheel_radius" value="${props['wheel_radius']}" />
+    <xacro:property name="wheel_length" value="${props['wheel_length']}" />
+    <xacro:property name="wheel_mass" value="${props['wheel_mass']}" />
     <xacro:macro name="link_wheel" params="name">
         <link name="${name}">
             <inertial>
-              <mass value="0.2"/>
+              <mass value="${wheel_mass}"/>
               <origin rpy="0 1.5707 1.5707" xyz="0 0 0"/>
               <inertia ixx="0.000526666666667" ixy="0" ixz="0" iyy="0.000526666666667" iyz="0" izz="0.001"/>
@@ -11,5 +16,5 @@
               <origin rpy="0 1.5707 1.5707" xyz="0 0 0"/>
               <geometry>
-                <cylinder length="0.04" radius="0.1"/>
+                <cylinder length="${wheel_length}" radius="${wheel_radius}"/>
               </geometry>
             </collision>
@@ -17,5 +22,5 @@
               <origin rpy="0 1.5707 1.5707" xyz="0 0 0"/>
               <geometry>
-                <cylinder length="0.04" radius="0.1"/>
+                <cylinder length="${wheel_length}" radius="${wheel_radius}"/>
               </geometry>
             </visual>

Commit message: reomoved comments

File: diff_drive/urdf/ddrive.urdf.xacro (robot description, xacro)
@@ -10,17 +10,4 @@
 <xacro:property name="height" value="${props['height']}" />
 <xacro:property name="caster_radius" value="${props['caster_radius']}" />
-  <!-- <link name="World">
-      <visual>
-      <origin rpy="0 0 0" xyz="0 0 0"/>
-      <geometry>
-        <box size="${width} ${length} ${height}"/>
-      </geometry>
-    </visual>
-  </link>
-  <joint name="World_Joint" type="fixed">
-  <origin rpy="0 0 0" xyz="0 0 0"/>
-  <child link="link_chassis"/>
-  <parent link="World"/>
-  </joint> -->
 <link name="dummy">
    </link>

Commit message: multiple changes some have to go away

File: diff_drive/urdf/ddrive.urdf.xacro (robot description, xacro)
@@ -16,11 +16,18 @@
      <child link="link_chassis"/>
    </joint>
+<!-- width**2 = 0.25
+d**2 = 0.09
+height**2 = 0.0049
+5/12 = 2.4
+width + d * mass/12 = 0.816
+d + h * mass/12 = 0.22776
+w+ h * mass/12 =  0.61176 -->
   <link name="link_chassis">
     <!-- pose and inertial -->
-    <pose>0 0 0.1 0 0 0</pose>
+    <pose>0 0 0.0 0 0 0</pose>
     <inertial>
-      <mass value="5"/>
-      <origin rpy="0 0 0" xyz="0 0 0.1"/>
-      <inertia ixx="0.0395416666667" ixy="0" ixz="0" iyy="0.106208333333" iyz="0" izz="0.106208333333"/>
+      <mass value="0.5"/>
+      <origin rpy="0 0 0" xyz="0 0 0"/>
+      <inertia ixx="0.022776" ixy="0" ixz="0" iyy="0.061176" iyz="0" izz="0.0816"/>
     </inertial>
     <!-- body -->
@@ -85,6 +92,6 @@
   </link>
   <xacro:link_wheel name="link_right_wheel" />
-  <xacro:joint_wheel name="joint_right_wheel" child="link_right_wheel" origin_xyz="-0.05 0.20 0" />
+  <xacro:joint_wheel name="joint_right_wheel" child="link_right_wheel" origin_xyz="-0.2 0.20 0" />
   <xacro:link_wheel name="link_left_wheel" />
-  <xacro:joint_wheel name="joint_left_wheel" child="link_left_wheel" origin_xyz="-0.05 -0.20 0" />
+  <xacro:joint_wheel name="joint_left_wheel" child="link_left_wheel" origin_xyz="-0.2 -0.20 0" />
 </robot>
