Commit message: added function of cylynder inertia

File: diff_drive/urdf/ddrive.urdf.xacro (robot description, xacro)
@@ -16,11 +16,4 @@
      <child link="link_chassis"/>
    </joint>
-<!-- width**2 = 0.25
-d**2 = 0.09
-height**2 = 0.0049
-5/12 = 2.4
-width + d * mass/12 = 0.816
-d + h * mass/12 = 0.22776
-w+ h * mass/12 =  0.61176 -->
   <link name="link_chassis">
     <!-- pose and inertial -->
@@ -30,4 +23,5 @@
       <origin rpy="0 0 0" xyz="0 0 0"/>
       <inertia ixx="0.022776" ixy="0" ixz="0" iyy="0.061176" iyz="0" izz="0.0816"/>
+      <!-- <xacro:cube_inertia mass="0.5" h="${width}" w="${length}" d="${height}" /> -->
     </inertial>
     <!-- body -->
@@ -50,14 +44,4 @@
         <sphere radius="${caster_radius}"/>
       </geometry>
-      <surface>
-        <friction>
-          <ode>
-            <mu>0</mu>
-            <mu2>0</mu2>
-            <slip1>1.0</slip1>
-            <slip2>1.0</slip2>
-          </ode>
-        </friction>
-      </surface>
     </collision>
     <visual name="caster_down_visual">
@@ -73,14 +57,4 @@
         <sphere radius="${caster_radius}"/>
       </geometry>
-      <surface>
-        <friction>
-          <ode>
-            <mu>0</mu>
-            <mu2>0</mu2>
-            <slip1>1.0</slip1>
-            <slip2>1.0</slip2>
-          </ode>
-        </friction>
-      </surface>
     </collision>
     <visual name="caster_up_visual">

File: diff_drive/urdf/macros.xacro (robot description, xacro)
@@ -8,10 +8,6 @@
     <xacro:macro name="link_wheel" params="name">
         <link name="${name}">
-            <inertial>
-              <mass value="${wheel_mass}"/>
-              <origin rpy="0 1.5707 1.5707" xyz="0 0 0"/>
-              <inertia ixx="0.000526666666667" ixy="0" ixz="0" iyy="0.000526666666667" iyz="0" izz="0.001"/>
-            </inertial>
-            <collision name="link_right_wheel_collision">
+              <xacro:cylinder_inertia mass="${wheel_mass}" r="${wheel_radius}" l="${wheel_length}"/>
+            <collision name="${name}__collision">
               <origin rpy="0 1.5707 1.5707" xyz="0 0 0"/>
               <geometry>
@@ -38,7 +34,27 @@
     </xacro:macro>
     <xacro:macro name="cylinder_inertia" params="mass r l">
-      <inertia  ixx="${mass*(3*r*r+l*l)/12}" ixy = "0" ixz = "0"
-                iyy="${mass*(3*r*r+l*l)/12}" iyz = "0"
-                izz="${mass*(r*r)/2}" />
+      <inertial>
+        <mass value="${mass}"/>
+        <origin rpy="0 1.5707 1.5707" xyz="0 0 0"/>
+        <inertia  ixx="${mass*(3*r*r+l*l)/12}" ixy = "0" ixz = "0"
+                  iyy="${mass*(3*r*r+l*l)/12}" iyz = "0"
+                  izz="${mass*(r*r)/2}" />
+      </inertial>
+    </xacro:macro>
+    <xacro:macro name="cube_inertia" params="mass h w d ">
+      <inertia  ixx="${mass*(w*w + d*d)/12}" ixy = "0" ixz = "0"
+                iyy="${mass*(h*h + d*d)/12}" iyz = "0"
+                izz="${mass*(h*h + w*w)/12}" />
     </xacro:macro>
 </robot>
+<!-- cube inertia  -->
+<!-- 2.88*(0.3*0.3+0.07*0.07)/12 xx -->
+<!-- 2.88*(0.5*0.5+0.07*0.07)/12 yy -->
+<!-- 2.88*(0.5*0.5+0.3*0.3)/12   zz-->
+<!-- cylinder inertia  -->
+<!-- wheel_radius: 0.1 -->
+<!-- wheel_length: 0.04 -->
+<!-- wheel_mass : 0.2 -->
+<!-- 0.2*(3*0.1*0.1+0.04*0.04)/12 -->
+<!-- 0.2*(3*0.1*0.1+0.04*0.04)/12 -->
+<!-- 0.2*(0.1*0.1)/2 -->

Commit message: added caster function

File: diff_drive/urdf/ddrive.urdf.xacro (robot description, xacro)
@@ -38,30 +38,7 @@
       <material name="blue"/>
     </visual>
-    <!-- caster down -->
-    <collision name="caster_down_collision">
-      <origin rpy=" 0 0 0" xyz="0.35 0 -0.05"/>
-      <geometry>
-        <sphere radius="${caster_radius}"/>
-      </geometry>
-    </collision>
-    <visual name="caster_down_visual">
-      <origin rpy=" 0 0 0" xyz="0.2 0 -0.05"/>
-      <geometry>
-        <sphere radius="${caster_radius}"/>
-      </geometry>
-    </visual>
-    <!-- caster up -->
-    <collision name="caster_up_collision">
-      <origin rpy=" 0 0 0" xyz="0.35 0 0.05"/>
-      <geometry>
-        <sphere radius="${caster_radius}"/>
-      </geometry>
-    </collision>
-    <visual name="caster_up_visual">
-      <origin rpy=" 0 0 0" xyz="0.2 0 0.05"/>
-      <geometry>
-        <sphere radius="${caster_radius}"/>
-      </geometry>
-    </visual>
+    <!-- caster -->
+    <xacro:caster name="caster_down" z="-0.05" />
+    <xacro:caster name="caster_up"   z=" 0.05" />
   </link>
   <xacro:link_wheel name="link_right_wheel" />

File: diff_drive/urdf/macros.xacro (robot description, xacro)
@@ -6,4 +6,5 @@
     <xacro:property name="wheel_length" value="${props['wheel_length']}" />
     <xacro:property name="wheel_mass" value="${props['wheel_mass']}" />
+    <xacro:property name="caster_radius" value="${props['caster_radius']}" />
     <xacro:macro name="link_wheel" params="name">
         <link name="${name}">
@@ -33,4 +34,18 @@
       </joint>
     </xacro:macro>
+    <xacro:macro name="caster" params="name z" >
+        <collision name="${name}_collision">
+        <origin rpy=" 0 0 0" xyz="0.35 0 ${z}"/>
+        <geometry>
+          <sphere radius="${caster_radius}"/>
+        </geometry>
+      </collision>
+      <visual name="${name}_visual">
+        <origin rpy=" 0 0 0" xyz="0.2 0 ${z}"/>
+        <geometry>
+          <sphere radius="${caster_radius}"/>
+        </geometry>
+      </visual>
+    </xacro:macro>
     <xacro:macro name="cylinder_inertia" params="mass r l">
       <inertial>

Commit message: moves inertia to macros function

File: diff_drive/urdf/ddrive.urdf.xacro (robot description, xacro)
@@ -19,10 +19,5 @@
     <!-- pose and inertial -->
     <pose>0 0 0.0 0 0 0</pose>
-    <inertial>
-      <mass value="0.5"/>
-      <origin rpy="0 0 0" xyz="0 0 0"/>
-      <inertia ixx="0.022776" ixy="0" ixz="0" iyy="0.061176" iyz="0" izz="0.0816"/>
-      <!-- <xacro:cube_inertia mass="0.5" h="${width}" w="${length}" d="${height}" /> -->
-    </inertial>
+    <xacro:cube_inertia mass="0.5" h="${width}" w="${length}" d="${height}" />
     <!-- body -->
     <collision name="collision_chassis">

File: diff_drive/urdf/macros.xacro (robot description, xacro)
@@ -58,7 +58,12 @@
     </xacro:macro>
     <xacro:macro name="cube_inertia" params="mass h w d ">
-      <inertia  ixx="${mass*(w*w + d*d)/12}" ixy = "0" ixz = "0"
-                iyy="${mass*(h*h + d*d)/12}" iyz = "0"
-                izz="${mass*(h*h + w*w)/12}" />
+        <inertial>
+          <mass value="0.5"/>
+          <origin rpy="0 0 0" xyz="0 0 0"/>
+          <inertia ixx="0.022776" ixy="0" ixz="0" iyy="0.061176" iyz="0" izz="0.0816"/>
+          <!-- <inertia  ixx="${mass*(w*w + d*d)/12}" ixy = "0" ixz = "0"
+                    iyy="${mass*(h*h + d*d)/12}" iyz = "0"
+                    izz="${mass*(h*h + w*w)/12}" /> -->
+        </inertial>
     </xacro:macro>
 </robot>

Commit message: fixed bug with base frame

File: diff_drive/urdf/ddrive.urdf.xacro (robot description, xacro)
@@ -10,8 +10,8 @@
 <xacro:property name="height" value="${props['height']}" />
 <xacro:property name="caster_radius" value="${props['caster_radius']}" />
-<link name="dummy">
+<link name="odom">
    </link>
   <joint name="dummy_joint" type="fixed">
-     <parent link="dummy"/>
+     <parent link="odom"/>
      <child link="link_chassis"/>
    </joint>
